File: resources/35um/Hotplate-100_100_4_8ohm.35um.kicad_pcb (KiCad board)
At the start: 2 copper layers, 100 x 100 mm, 7 parts, among them J1 Hotplate_Power_Connection, J2 Hotplate_Power_Connection

Commit message: Replaced obsolete 25mm thermal fuse footprint with new 35mm thermal fuse footprint.
Parts:
- F1: footprint blg:Thermal Fuse, Front, 25mm -> blg:Thermal Fuse, SN100C, Front, 35mm
Routing:
- net Net-(J2-Pin_1): track 3304.6 -> 3283.8 mm
- net Net-(J1-Pin_1): track 3263.2 -> 3282.3 mm
Other:
- board text added: "Cold Resistance: 2.739Ω Hot Resistance: 4.798Ω Voltage: 24V Power: 120W Generated: 20251229-234414"
- board text removed: "Cold Resistance: 2.740Ω Hot Resistance: 4.800Ω Voltage: 24V Power: 120W Generated: 20250914-162736"
